Commit message: add imu offset

File: src/ros_pathfinder/urdf/pathfinder.urdf.xacro (robot description, xacro)
@@ -9,5 +9,5 @@
   <xacro:property name="wheel_separation" value="0.24"/>
   <!-- TODO: measure imu to base link values. -->
-  <xacro:property name="imu_x" value="0.0"/>
+  <xacro:property name="imu_x" value="0.195"/>
   <xacro:property name="imu_y" value="0.0"/>
   <xacro:property name="imu_z" value="0.05"/>

Commit message: broadcast odom->base_link transform

File: src/ros_pathfinder/urdf/pathfinder.urdf.xacro (robot description, xacro)
@@ -1,15 +1,13 @@
 <?xml version="1.0"?>
 <robot xmlns:xacro="http://www.ros.org/wiki/xacro" name="pathfinder">
-  <!-- TODO: confirm values here -->
-  <xacro:property name="base_length" value="0.25"/>
-  <xacro:property name="base_width" value="0.20"/>
+  <xacro:property name="base_length" value="0.604"/>
+  <xacro:property name="base_width" value="0.451"/>
   <xacro:property name="base_height" value="0.08"/>
   <xacro:property name="wheel_radius" value="0.1016"/>
   <xacro:property name="wheel_width" value="0.04"/>
   <xacro:property name="wheel_separation" value="0.24"/>
-  <!-- TODO: measure imu to base link values. -->
   <xacro:property name="imu_x" value="0.195"/>
   <xacro:property name="imu_y" value="0.0"/>
-  <xacro:property name="imu_z" value="0.05"/>
+  <xacro:property name="imu_z" value="0.0"/>
   <!-- TODO: confirm lidar transform values after statically mounting it -->
   <xacro:property name="laser_x" value="0.32"/>

Commit message: update urdf values

File: src/ros_pathfinder/urdf/pathfinder.urdf.xacro (robot description, xacro)
@@ -4,7 +4,11 @@
   <xacro:property name="base_width" value="0.451"/>
   <xacro:property name="base_height" value="0.08"/>
+  <xacro:property name="base_link_from_rear" value="0.127"/>
   <xacro:property name="wheel_radius" value="0.1016"/>
   <xacro:property name="wheel_width" value="0.04"/>
-  <xacro:property name="wheel_separation" value="0.24"/>
+  <xacro:property
+    name="wheel_separation"
+    value="${base_width + wheel_width}"
+  />
   <xacro:property name="imu_x" value="0.195"/>
   <xacro:property name="imu_y" value="0.0"/>
@@ -27,5 +31,8 @@
   <link name="base_link">
     <visual>
-      <origin xyz="0 0 ${base_height / 2.0}" rpy="0 0 0"/>
+      <origin
+        xyz="${base_length / 2.0 - base_link_from_rear} 0 ${base_height / 2.0}"
+        rpy="0 0 0"
+      />
       <geometry>
         <box size="${base_length} ${base_width} ${base_height}"/>
@@ -34,5 +41,8 @@
     </visual>
     <collision>
-      <origin xyz="0 0 ${base_height / 2.0}" rpy="0 0 0"/>
+      <origin
+        xyz="${base_length / 2.0 - base_link_from_rear} 0 ${base_height / 2.0}"
+        rpy="0 0 0"
+      />
       <geometry>
         <box size="${base_length} ${base_width} ${base_height}"/>
